File: Schematic/Arduino_MEGA_2560-Rev3.sch (KiCad schematic (older format))
At the start: 103 parts, among them IC1 NCP1117ST50T3G, IC3 ATMEGA2560-16AU, IC4 ATMEGA16U2-MU, IC6 LP2985-33DBVR, IC7 LMV358IDGKR, T1 FDN340P, X1 POWERSUPPLY_DC21MMX, X2 USB-B_TH, Y1 CSTCE16M0V53-R0 16MHZ, Y2 16MHz

Commit message: Added Button Game Schematic
Parts:
- added D?: LED_RGB, symbol Device:LED_RGB
- added R?: R, symbol Device:R
- added SW?: SW_Push, symbol Switch:SW_Push
Connections:
- net labels added: 23, 24, 25, 26, 27
- wire segments 570 -> 587
Other:
- note added: "Button Game\n\n\n"

Commit message: Added Simon Says Schematic
Parts:
- added D? (x4): LED_ALT, symbol Device:LED_ALT
- added R? (x4): 300R, symbol Device:R
- added R? (x4): 4.7K, symbol Device:R
- added SW? (x4): SW_Push, symbol Switch:SW_Push
Connections:
- net labels added: 28, 29, 30
- wire segments 587 -> 627
Other:
- note added: "Simon Says Game\n\n"

Commit message: Schematic Annotated
Parts:
- R17: renamed from R?; value R -> 4.7k
- gave numbers to parts that had none: 62
Other:
- note added: "Blue\n"
- note added: "Green\n"
- note added: "Red\n"
- note added: "Yellow\n"
