File: Schematic/Arduino_MEGA_2560-Rev3.sch (KiCad schematic (older format))
At the start: 122 parts, among them IC1 NCP1117ST50T3G, IC3 ATMEGA2560-16AU, IC4 ATMEGA16U2-MU, IC6 LP2985-33DBVR, IC7 LMV358IDGKR, Q1 2N2222, Q2 2N2222, Q3 2N2222, Q4 2N2222, SW1 SW_Push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

Commit message: Added Completion Indication to Schematic
Parts:
- added D? (x3): LED_ALT, symbol Device:LED_ALT
- added R? (x3): 4.7K, symbol Device:R
Connections:
- net labels added: 38, 39, 40
- wire segments 627 -> 639
Other:
- note added: "Completion\n\n"

Commit message: Schematic
Parts:
- added D? (x2): LED_ALT, symbol Device:LED_ALT
- added R? (x2): 4.7K, symbol Device:R
- gave numbers to parts that had none: 6
- renumbered 4.7K to 4.7K1
Connections:
- net labels added: 41, 42
- wire segments 639 -> 647
Other:
- note added: "Red"
Changed lines of the file:
@@
 	5400 1500 5400 11300
 $Comp
-L Device:R_POT 4.7K
+L Device:R_POT 4.7K1
 U 1 1 5DDD3DFD
 P 19150 13850
-F 0 "4.7K" V 19150 13950 50  0000 R CNN
+F 0 "4.7K1" V 19150 13950 50  0000 R CNN
 F 1 "R_POT" V 19050 13950 50  0000 R CNN
 F 2 "" H 19150 13850 50  0001 C CNN
@@
 Yellow\n
 $Comp
+L Device:LED_ALT D42
+U 1 1 5CF34215
+P 21750 18300
+F 0 "D42" V 21788 18182 50  0000 R CNN
+F 1 "LED_ALT" V 21697 18182 50  0000 R CNN
+F 2 "" H 21750 18300 50  0001 C CNN
+F 3 "~" H 21750 18300 50  0001 C CNN
+	1    21750 18300
+	0    -1   -1   0
+$EndComp
+$Comp
+L Device:LED_ALT D43
+U 1 1 5CFA4E91
+P 22250 18300
+F 0 "D43" V 22288 18182 50  0000 R CNN
+F 1 "LED_ALT" V 22197 18182 50  0000 R CNN
+F 2 "" H 22250 18300 50  0001 C CNN
+F 3 "~" H 22250 18300 50  0001 C CNN
+	1    22250 18300
+	0    -1   -1   0
+$EndComp
+$Comp
+L Device:LED_ALT D44
+U 1 1 5D01598C
+P 22750 18300
+F 0 "D44" V 22788 18182 50  0000 R CNN
+F 1 "LED_ALT" V 22697 18182 50  0000 R CNN
+F 2 "" H 22750 18300 50  0001 C CNN
+F 3 "~" H 22750 18300 50  0001 C CNN
+	1    22750 18300
+	0    -1   -1   0
+$EndComp
+Wire Wire Line
+	21750 18150 21750 18050
+Wire Wire Line
+	22250 18150 22250 18050
+Wire Wire Line
+	22750 18150 22750 18050
+$Comp
+L Device:R R18
+U 1 1 5D32C8A2
+P 21750 17900
+F 0 "R18" V 21650 17900 50  0000 C CNN
+F 1 "4.7K" V 21750 17900 50  0000 C CNN
+F 2 "" V 21680 17900 50  0001 C CNN
+F 3 "~" H 21750 17900 50  0001 C CNN
+	1    21750 17900
+	1    0    0    -1
+$EndComp
+$Comp
+L Device:R R19
+U 1 1 5D39E312
+P 22250 17900
+F 0 "R19" V 22150 17900 50  0000 C CNN
+F 1 "4.7K" V 22250 17900 50  0000 C CNN
+F 2 "" V 22180 17900 50  0001 C CNN
+F 3 "~" H 22250 17900 50  0001 C CNN
+	1    22250 17900
+	1    0    0    -1
+$EndComp
+$Comp
+L Device:R R20
+U 1 1 5D40F7A4
+P 22750 17900
+F 0 "R20" V 22650 17900 50  0000 C CNN
+F 1 "4.7K" V 22750 17900 50  0000 C CNN
+F 2 "" V 22680 17900 50  0001 C CNN
+F 3 "~" H 22750 17900 50  0001 C CNN
+	1    22750 17900
+	1    0    0    -1
+$EndComp
+Wire Wire Line
+	21750 17750 21750 17650
+Wire Wire Line
+	22250 17750 22250 17650
+Wire Wire Line
+	22750 17750 22750 17650
+Text GLabel 21750 17650 1    50   Input ~ 0
+38
+Text GLabel 22250 17650 1    50   Input ~ 0
+39
+Text GLabel 22750 17650 1    50   Input ~ 0
+40
+Wire Wire Line
+	21750 18550 21750 18450
+Wire Wire Line
+	22250 18550 22250 18450
+Wire Wire Line
+	22750 18550 22750 18450
+Wire Wire Line
+	22750 18550 22250 18550
+Connection ~ 22250 18550
+Wire Wire Line
+	22250 18550 21750 18550
+Wire Wire Line
+	22750 18550 22750 18700
+$Comp
+L power:GND #PWR020
+U 1 1 5D9DB52F
+P 22750 18700
+F 0 "#PWR020" H 22750 18450 50  0001 C CNN
+F 1 "GND" H 22900 18650 50  0000 C CNN
+F 2 "" H 22750 18700 50  0001 C CNN
+F 3 "" H 22750 18700 50  0001 C CNN
+	1    22750 18700
+	1    0    0    -1
+$EndComp
+Wire Notes Line
+	21250 17200 21250 19200
+Text Notes 23800 19500 2    254  ~ 0
+Completion\n\n
+Wire Notes Line
+	24200 19200 24200 17200
+Text GLabel 6200 7450 0    50   Input ~ 0
+25
+Text GLabel 7700 7350 2    50   Input ~ 0
+26
+Text GLabel 6200 7350 0    50   Input ~ 0
+27
+Text GLabel 7700 7250 2    50   Input ~ 0
+28
+Text GLabel 6200 7250 0    50   Input ~ 0
+29
+Text GLabel 7700 7150 2    50   Input ~ 0
+30
+$Comp
 L Device:LED_ALT D?
-U 1 1 5CF34215
-P 21800 18300
-F 0 "D?" V 21838 18182 50  0000 R CNN
-F 1 "LED_ALT" V 21747 18182 50  0000 R CNN
-F 2 "" H 21800 18300 50  0001 C CNN
-F 3 "~" H 21800 18300 50  0001 C CNN
-	1    21800 18300
+U 1 1 5E1929DC
+P 23250 18300
+F 0 "D?" V 23288 18182 50  0000 R CNN
+F 1 "LED_ALT" V 23197 18182 50  0000 R CNN
+F 2 "" H 23250 18300 50  0001 C CNN
+F 3 "~" H 23250 18300 50  0001 C CNN
+	1    23250 18300
 	0    -1   -1   0
 $EndComp
 $Comp
 L Device:LED_ALT D?
-U 1 1 5CFA4E91
-P 22300 18300
-F 0 "D?" V 22338 18182 50  0000 R CNN
-F 1 "LED_ALT" V 22247 18182 50  0000 R CNN
-F 2 "" H 22300 18300 50  0001 C CNN
-F 3 "~" H 22300 18300 50  0001 C CNN
-	1    22300 18300
-	0    -1   -1   0
-$EndComp
-$Comp
-L Device:LED_ALT D?
-U 1 1 5D01598C
-P 22800 18300
-F 0 "D?" V 22838 18182 50  0000 R CNN
-F 1 "LED_ALT" V 22747 18182 50  0000 R CNN
-F 2 "" H 22800 18300 50  0001 C CNN
-F 3 "~" H 22800 18300 50  0001 C CNN
-	1    22800 18300
-	0    -1   -1   0
-$EndComp
-Wire Wire Line
-	21800 18150 21800 18050
-Wire Wire Line
-	22300 18150 22300 18050
-Wire Wire Line
-	22800 18150 22800 18050
+U 1 1 5E1929E3
+P 23750 18300
+F 0 "D?" V 23788 18182 50  0000 R CNN
+F 1 "LED_ALT" V 23697 18182 50  0000 R CNN
+F 2 "" H 23750 18300 50  0001 C CNN
+F 3 "~" H 23750 18300 50  0001 C CNN
+	1    23750 18300
+	0    -1   -1   0
+$EndComp
+Wire Wire Line
+	23250 18150 23250 18050
+Wire Wire Line
+	23750 18150 23750 18050
 $Comp
 L Device:R R?
-U 1 1 5D32C8A2
-P 21800 17900
-F 0 "R?" V 21700 17900 50  0000 C CNN
-F 1 "4.7K" V 21800 17900 50  0000 C CNN
-F 2 "" V 21730 17900 50  0001 C CNN
-F 3 "~" H 21800 17900 50  0001 C CNN
-	1    21800 17900
+U 1 1 5E1929EC
+P 23250 17900
+F 0 "R?" V 23150 17900 50  0000 C CNN
+F 1 "4.7K" V 23250 17900 50  0000 C CNN
+F 2 "" V 23180 17900 50  0001 C CNN
+F 3 "~" H 23250 17900 50  0001 C CNN
+	1    23250 17900
 	1    0    0    -1
 $EndComp
 $Comp
 L Device:R R?
-U 1 1 5D39E312
-P 22300 17900
-F 0 "R?" V 22200 17900 50  0000 C CNN
-F 1 "4.7K" V 22300 17900 50  0000 C CNN
-F 2 "" V 22230 17900 50  0001 C CNN
-F 3 "~" H 22300 17900 50  0001 C CNN
-	1    22300 17900
-	1    0    0    -1
-$EndComp
-$Comp
-L Device:R R?
-U 1 1 5D40F7A4
-P 22800 17900
-F 0 "R?" V 22700 17900 50  0000 C CNN
-F 1 "4.7K" V 22800 17900 50  0000 C CNN
-F 2 "" V 22730 17900 50  0001 C CNN
-F 3 "~" H 22800 17900 50  0001 C CNN
-	1    22800 17900
-	1    0    0    -1
-$EndComp
-Wire Wire Line
-	21800 17750 21800 17650
-Wire Wire Line
-	22300 17750 22300 17650
-Wire Wire Line
-	22800 17750 22800 17650
-Text GLabel 21800 17650 1    50   Input ~ 0
-38
-Text GLabel 22300 17650 1    50   Input ~ 0
-39
-Text GLabel 22800 17650 1    50   Input ~ 0
-40
-Wire Wire Line
-	21800 18550 21800 18450
-Wire Wire Line
-	22300 18550 22300 18450
-Wire Wire Line
-	22800 18550 22800 18450
-Wire Wire Line
-	22800 18550 22300 18550
-Connection ~ 22300 18550
-Wire Wire Line
-	22300 18550 21800 18550
-Wire Wire Line
-	22300 18550 22300 18700
-$Comp
-L power:GND #PWR?
-U 1 1 5D9DB52F
-P 22300 18700
-F 0 "#PWR?" H 22300 18450 50  0001 C CNN
-F 1 "GND" H 22450 18650 50  0000 C CNN
-F 2 "" H 22300 18700 50  0001 C CNN
-F 3 "" H 22300 18700 50  0001 C CNN
-	1    22300 18700
-	1    0    0    -1
-$EndComp
-Wire Notes Line
-	21250 17200 21250 19200
-Text Notes 23450 19500 2    254  ~ 0
-Completion\n\n
-Wire Notes Line
-	23450 19200 23450 17200
-Wire Notes Line
-	21250 17200 23450 17200
-Wire Notes Line
-	21250 19200 23450 19200
+U 1 1 5E1929F3
+P 23750 17900
+F 0 "R?" V 23650 17900 50  0000 C CNN
+F 1 "4.7K" V 23750 17900 50  0000 C CNN
+F 2 "" V 23680 17900 50  0001 C CNN
+F 3 "~" H 23750 17900 50  0001 C CNN
+	1    23750 17900
+	1    0    0    -1
+$EndComp
+Wire Wire Line
+	23250 17750 23250 17650
+Wire Wire Line
+	23750 17750 23750 17650
+Text GLabel 23250 17650 1    50   Input ~ 0
+41
+Text GLabel 23750 17650 1    50   Input ~ 0
+42
+Wire Wire Line
+	22750 18550 23250 18550
+Wire Wire Line
+	23250 18550 23250 18450
+Connection ~ 22750 18550
+Wire Wire Line
+	23250 18550 23750 18550
+Wire Wire Line
+	23750 18550 23750 18450
+Connection ~ 23250 18550
+Text Notes 22350 17450 2    50   ~ 0
+Green\n
+Text Notes 23550 17450 2    50   ~ 0
+Red
+Wire Notes Line
+	21250 17200 24200 17200
+Wire Notes Line
+	21250 19200 24200 19200
 $EndSCHEMATC
